File: SPR5-HQ/hardware/KiCad/original/PowerSupply_SPR5HQ_original_1Layer_THT.kicad_pcb (KiCad board)
At the start: 2 copper layers, 120 x 87 mm, 62 parts, among them J1 Screw_Terminal_01x02, J2 Screw_Terminal_01x02, J3 Screw_Terminal_01x02, J4 Screw_Terminal_01x02, U1 LM338, U2 LM338

Commit message: Add files via upload
Routing:
- net /adj_1: track 110.2 -> 109.1 mm
