File: SPR5-HQ/hardware/KiCad/original V2/PowerSupply_SPR5HQ_original_1Layer_THT_v2.kicad_pcb (KiCad board)
At the start: 2 copper layers, 120 x 87 mm, 68 parts, among them J1 Screw_Terminal_01x02, J2 Screw_Terminal_01x02, J3 Screw_Terminal_01x02, J4 Screw_Terminal_01x02, U1 LM338, U2 LM338

Commit message: Add files via upload
Parts:
- D10, D12: footprint analoghifi:D_DO-41_SOD81_P10.16mm_Horizontal_minSilk -> analoghifi:D_DO-41_SOD81_short_P9.0mm_Horiz_minSilk
- R1, R2: footprint analoghifi:R_Axial_DIN0207_L6.3mm_D2.5mm_P10.16mm_Horizontal_minSilk -> analoghifi:R_Axial_Short_L6.3mm_D2.5mm_P9.0mm_Horiz_minSilk
- moved D10 1.54 mm to (159.5, 80.0)
- moved D12 1.54 mm to (159.5, 127.0)
- moved R1 1.54 mm to (159.5, 83.0)
- moved R2 1.54 mm to (159.5, 124.0)
- moved C19 1.06 mm to (155.2, 133.4)
- moved C20 1.06 mm to (151.5, 112.2)
- moved C8 1.06 mm to (155.2, 73.6)
- moved C9 1.06 mm to (155.2, 91.1)
- moved L1 1.06 mm to (153.5, 79.8)
- moved L2 1.06 mm to (153.5, 127.2)
- moved C11 0.50 mm to (167.5, 75.8)
- moved C22 0.50 mm to (167.5, 131.2)
- moved D11 0.50 mm to (123.8, 125.8)
Routing:
- net /pos2_r: track 0.00 -> 6.63 mm
- net /adj_1: track 48.3 -> 44.9 mm
- net /adj_2: track 48.3 -> 49.7 mm
